File: AB2-K03D - Models/AB2-K03D - Models.sch (KiCad schematic (older format))
At the start: 7 parts, among them X1 AB2_AKZ500_02

Commit message: AB2-K03D: add lqfp 60 pin render problems
Parts:
- removed C1: 0.1u, symbol AB2_C
- removed C2: 0.47u, symbol AB2_C
- removed DRV1, DRV2: AB2_DRV8828/9, ~, symbol AB2_DRV8828/9
- removed HDR1: AB2_HDR06-1_SBW, ~, symbol AB2_HDR06-1_SBW
- removed MSP1: MSP430F5510_48, ~, symbol MSP430F5510_48
- removed X1: AB2_AKZ500_02, ~, symbol AB2_AKZ500_02
Connections:
- net labels removed: AB2_GND, AB2_MSP3V6, AB2_PRG3V6, AVCC1, D+, D-, PUR, RST/NMI/SBWTDIO, RXD, TEST/SBWTCK, TXD, VBUS, VCORE, VUSB
- wire segments 11 -> 0
