File: AB2-K03D - Models/AB2-K03D - Models.kicad_pcb (KiCad board)
At the start: 2 copper layers, 87 parts, among them X1 AB2_AKZ500_02

Commit message: AB2-K03D: initial commit of 3d model proj visualizer
Parts:
- removed C1: 0.1u, AB2_0805
- removed C2: 0.47u, AB2_0805
- removed DRV1, DRV2: AB2_DRV8828/9, AB2_TSSOP28-PWP2
- removed MSP1: MSP430F5510_48, AB2_LQFP48
- removed X1: AB2_AKZ500_02, AB2_AKZ500_02
- added AB2_HDR_M07-2V: VAL**, AB2_HDR_M07-2V, F.Cu at (96.5, 47.0)
- added AB2_HDR_M08-2V: VAL**, AB2_HDR_M08-2V, F.Cu at (97.8, 52.1)
- added AB2_HDR_M09-2V: VAL**, AB2_HDR_M09-2V, F.Cu at (99.1, 57.1)
- added AB2_HDR_M10-2V: VAL**, AB2_HDR_M10-2V, F.Cu at (100.3, 62.2)
- added AB2_HDR_M11-2V: VAL**, AB2_HDR_M11-2V, F.Cu at (101.6, 67.3)
- added AB2_HDR_M12-2V: VAL**, AB2_HDR_M12-2V, F.Cu at (102.9, 72.4)
- added AB2_HDR_M13-2V: VAL**, AB2_HDR_M13-2V, F.Cu at (104.1, 77.5)
- added AB2_HDR_M14-2V: VAL**, AB2_HDR_M14-2V, F.Cu at (105.4, 82.5)
- added AB2_HDR_M15-2V: VAL**, AB2_HDR_M15-2V, F.Cu at (106.7, 87.6)
- added AB2_HDR_M16-2V: VAL**, AB2_HDR_M16-2V, F.Cu at (108.0, 92.7)
- added AB2_HDR_M17-2V: VAL**, AB2_HDR_M17-2V, F.Cu at (109.2, 97.8)
- added AB2_HDR_M18-2V: VAL**, AB2_HDR_M18-2V, F.Cu at (110.5, 102.9)
- added AB2_HDR_M19-2V: VAL**, AB2_HDR_M19-2V, F.Cu at (111.8, 108.0)
- added AB2_HDR_M20-2V: VAL**, AB2_HDR_M20-2V, F.Cu at (113.0, 113.0)
- added AB2_HDR_M21-2V: VAL**, AB2_HDR_M21-2V, F.Cu at (114.3, 118.1)
- added AB2_HDR_M22-2V: VAL**, AB2_HDR_M22-2V, F.Cu at (115.6, 123.2)
- added AB2_HDR_M23-2V: VAL**, AB2_HDR_M23-2V, F.Cu at (116.8, 128.3)
- added AB2_HDR_M24-2V: VAL**, AB2_HDR_M24-2V, F.Cu at (118.1, 133.3)
- added AB2_HDR_M25-2V: VAL**, AB2_HDR_M25-2V, F.Cu at (119.4, 138.4)
- moved AB2_HDR_M09-1V 287.2 mm to (25.4, 35.6)
- moved AB2_HDR_M12-1V 287.2 mm to (29.2, 43.2)
- moved AB2_HDR_M15-1V 287.2 mm to (33.0, 50.8)
- moved AB2_HDR_M18-1V 287.2 mm to (36.8, 58.4)
- moved HDR1 287.2 mm to (21.6, 27.9)
- moved AB2_HDR_M01-1V 287.2 mm to (15.2, 15.2)
- moved AB2_HDR_M02-1V 287.2 mm to (16.5, 17.8)
- moved AB2_HDR_M03-1V 287.2 mm to (17.8, 20.3)
- moved AB2_HDR_M04-1V 287.2 mm to (19.1, 22.9)
- moved AB2_HDR_M05-1V 287.2 mm to (20.3, 25.4)
- moved AB2_HDR_M07-1V 287.2 mm to (22.9, 30.5)
- moved AB2_HDR_M08-1V 287.2 mm to (24.1, 33.0)
- moved AB2_HDR_M10-1V 287.2 mm to (26.7, 38.1)
- moved AB2_HDR_M11-1V 287.2 mm to (27.9, 40.6)
- moved AB2_HDR_M13-1V 287.2 mm to (30.5, 45.7)
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
Commit message: AB2-K03D: add 805 caps and LQFP48 pin
Parts:
- added AB2_0805_C_125: VAL**, AB2_0805_C_125, F.Cu at (76.2, 20.3)
- added AB2_0805_C_60: VAL**, AB2_0805_C_60, F.Cu at (76.2, 15.2)
- added AB2_0805_C_80: VAL**, AB2_0805_C_80, F.Cu at (76.2, 17.8)
- added AB2_LQFP48: VAL**, AB2_LQFP48, F.Cu at (17.8, 279.4)
Changed lines of the file:
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@@
     (links 0)
     (no_connects 0)
-    (area 7.723012 12.0015 151.447501 233.743501)
+    (area 7.723012 12.0015 151.447501 284.669892)
     (thickness 1.6)
     (drawings 0)
     (tracks 0)
     (zones 0)
-    (modules 100)
+    (modules 104)
     (nets 6)
   )
@@
     )
   )
+  (module AB2_0805_C_60 (layer F.Cu)
+    (at 76.2 15.24)
+    (fp_text reference AB2_0805_C_60 (at 0 -1.27) (layer F.SilkS)
+      (effects (font (size 0.8128 0.8128) (thickness 0.0762)))
+    )
+    (fp_text value VAL** (at 0 1.27) (layer F.SilkS)
+      (effects (font (size 0.8128 0.8128) (thickness 0.0762)))
+    )
+    (fp_line (start -0.29972 0.59944) (end 0.29972 0.59944) (layer F.SilkS) (width 0.127))
+    (fp_line (start -0.29972 -0.59944) (end 0.29972 -0.59944) (layer F.SilkS) (width 0.127))
+    (pad 1 smd rect (at -0.9 0) (size 0.8 1.2)
+      (layers F.Cu F.Paste F.Mask)
+    )
+    (pad 2 smd rect (at 0.9 0) (size 0.8 1.2)
+      (layers F.Cu F.Paste F.Mask)
+    )
+    (model "../../../../Program Files (x86)/KiCad/share/3d_models/ab2_passive/AB2_0805_C_60.wrl"
+      (at (xyz 0 0 0))
+      (scale (xyz 0.3937 0.3937 0.3937))
+      (rotate (xyz 0 0 0))
+    )
+  )
+  (module AB2_0805_C_80 (layer F.Cu)
+    (at 76.2 17.78)
+    (fp_text reference AB2_0805_C_80 (at 0 -1.27) (layer F.SilkS)
+      (effects (font (size 0.8128 0.8128) (thickness 0.0762)))
+    )
+    (fp_text value VAL** (at 0 1.27) (layer F.SilkS)
+      (effects (font (size 0.8128 0.8128) (thickness 0.0762)))
+    )
+    (fp_line (start -0.29972 0.59944) (end 0.29972 0.59944) (layer F.SilkS) (width 0.127))
+    (fp_line (start -0.29972 -0.59944) (end 0.29972 -0.59944) (layer F.SilkS) (width 0.127))
+    (pad 1 smd rect (at -0.9 0) (size 0.8 1.2)
+      (layers F.Cu F.Paste F.Mask)
+    )
+    (pad 2 smd rect (at 0.9 0) (size 0.8 1.2)
+      (layers F.Cu F.Paste F.Mask)
+    )
+    (model "../../../../Program Files (x86)/KiCad/share/3d_models/ab2_passive/AB2_0805_C_80.wrl"
+      (at (xyz 0 0 0))
+      (scale (xyz 0.3937 0.3937 0.3937))
+      (rotate (xyz 0 0 0))
+    )
+  )
+  (module AB2_0805_C_125 (layer F.Cu)
+    (at 76.2 20.32)
+    (fp_text reference AB2_0805_C_125 (at 0 -1.27) (layer F.SilkS)
+      (effects (font (size 0.8128 0.8128) (thickness 0.0762)))
+    )
+    (fp_text value VAL** (at 0 1.27) (layer F.SilkS)
+      (effects (font (size 0.8128 0.8128) (thickness 0.0762)))
+    )
+    (fp_line (start -0.29972 0.59944) (end 0.29972 0.59944) (layer F.SilkS) (width 0.127))
+    (fp_line (start -0.29972 -0.59944) (end 0.29972 -0.59944) (layer F.SilkS) (width 0.127))
+    (pad 1 smd rect (at -0.9 0) (size 0.8 1.2)
+      (layers F.Cu F.Paste F.Mask)
+    )
+    (pad 2 smd rect (at 0.9 0) (size 0.8 1.2)
+      (layers F.Cu F.Paste F.Mask)
+    )
+    (model "../../../../Program Files (x86)/KiCad/share/3d_models/ab2_passive/AB2_0805_C_125.wrl"
+      (at (xyz 0 0 0))
+      (scale (xyz 0.3937 0.3937 0.3937))
+      (rotate (xyz 0 0 0))
+    )
+  )
+  (module AB2_LQFP48 (layer F.Cu)
+    (at 17.78 279.4)
+    (fp_text reference AB2_LQFP48 (at 0 -1.27) (layer F.SilkS)
+      (effects (font (size 0.8128 0.8128) (thickness 0.0762)))
+    )
+    (fp_text value VAL** (at 0 1.27) (layer F.SilkS)
+      (effects (font (size 0.8128 0.8128) (thickness 0.0762)))
+    )
+    (fp_circle (center -2.8 -2.8) (end -2.8 -3.1) (layer F.SilkS) (width 0.127))
+    (fp_line (start -3.5 -3.5) (end 3.5 -3.5) (layer F.SilkS) (width 0.127))
+    (fp_line (start 3.5 -3.5) (end 3.5 3.5) (layer F.SilkS) (width 0.127))
+    (fp_line (start 3.5 3.5) (end -3.5 3.5) (layer F.SilkS) (width 0.127))
+    (fp_line (start -3.5 3.5) (end -3.5 -3.5) (layer F.SilkS) (width 0.127))
+    (pad 6 smd rect (at -4.3 -0.25) (size 1.4 0.3)
+      (layers F.Cu F.Paste F.Mask)
+    )
+    (pad 5 smd rect (at -4.3 -0.75) (size 1.4 0.3)
+      (layers F.Cu F.Paste F.Mask)
+    )
+    (pad 4 smd rect (at -4.3 -1.25) (size 1.4 0.3)
+      (layers F.Cu F.Paste F.Mask)
+    )
+    (pad 3 smd rect (at -4.3 -1.75) (size 1.4 0.3)
+      (layers F.Cu F.Paste F.Mask)
+    )
+    (pad 2 smd rect (at -4.3 -2.25) (size 1.4 0.3)
+      (layers F.Cu F.Paste F.Mask)
+    )
+    (pad 1 smd rect (at -4.3 -2.75) (size 1.4 0.3)
+      (layers F.Cu F.Paste F.Mask)
+    )
+    (pad 7 smd rect (at -4.3 0.25) (size 1.4 0.3)
+      (layers F.Cu F.Paste F.Mask)
+    )
+    (pad 8 smd rect (at -4.3 0.75) (size 1.4 0.3)
+      (layers F.Cu F.Paste F.Mask)
+    )
+    (pad 9 smd rect (at -4.3 1.25) (size 1.4 0.3)
+      (layers F.Cu F.Paste F.Mask)
+    )
+    (pad 10 smd rect (at -4.3 1.75) (size 1.4 0.3)
+      (layers F.Cu F.Paste F.Mask)
+    )
+    (pad 11 smd rect (at -4.3 2.25) (size 1.4 0.3)
+      (layers F.Cu F.Paste F.Mask)
+    )
+    (pad 12 smd rect (at -4.3 2.75) (size 1.4 0.3)
+      (layers F.Cu F.Paste F.Mask)
+    )
+    (pad 13 smd rect (at -2.75 4.3) (size 0.3 1.4)
+      (layers F.Cu F.Paste F.Mask)
+    )
+    (pad 14 smd rect (at -2.25 4.3) (size 0.3 1.4)
+      (layers F.Cu F.Paste F.Mask)
+    )
+    (pad 15 smd rect (at -1.75 4.3) (size 0.3 1.4)
+      (layers F.Cu F.Paste F.Mask)
+    )
+    (pad 16 smd rect (at -1.25 4.3) (size 0.3 1.4)
+      (layers F.Cu F.Paste F.Mask)
+    )
+    (pad 17 smd rect (at -0.75 4.3) (size 0.3 1.4)
+      (layers F.Cu F.Paste F.Mask)
+    )
+    (pad 18 smd rect (at -0.25 4.3) (size 0.3 1.4)
+      (layers F.Cu F.Paste F.Mask)
+    )
+    (pad 19 smd rect (at 0.25 4.3) (size 0.3 1.4)
+      (layers F.Cu F.Paste F.Mask)
+    )
+    (pad 20 smd rect (at 0.75 4.3) (size 0.3 1.4)
+      (layers F.Cu F.Paste F.Mask)
+    )
+    (pad 21 smd rect (at 1.25 4.3) (size 0.3 1.4)
+      (layers F.Cu F.Paste F.Mask)
+    )
+    (pad 22 smd rect (at 1.75 4.3) (size 0.3 1.4)
+      (layers F.Cu F.Paste F.Mask)
+    )
+    (pad 23 smd rect (at 2.25 4.3) (size 0.3 1.4)
+      (layers F.Cu F.Paste F.Mask)
+    )
+    (pad 24 smd rect (at 2.75 4.3) (size 0.3 1.4)
+      (layers F.Cu F.Paste F.Mask)
+    )
+    (pad 25 smd rect (at 4.3 2.75) (size 1.4 0.3)
+      (layers F.Cu F.Paste F.Mask)
+    )
+    (pad 26 smd rect (at 4.3 2.25) (size 1.4 0.3)
+      (layers F.Cu F.Paste F.Mask)
+    )
+    (pad 27 smd rect (at 4.3 1.75) (size 1.4 0.3)
+      (layers F.Cu F.Paste F.Mask)
+    )
+    (pad 28 smd rect (at 4.3 1.25) (size 1.4 0.3)
+      (layers F.Cu F.Paste F.Mask)
+    )
+    (pad 29 smd rect (at 4.3 0.75) (size 1.4 0.3)
+      (layers F.Cu F.Paste F.Mask)
+    )
+    (pad 30 smd rect (at 4.3 0.25) (size 1.4 0.3)
+      (layers F.Cu F.Paste F.Mask)
+    )
+    (pad 31 smd rect (at 4.3 -0.25) (size 1.4 0.3)
+      (layers F.Cu F.Paste F.Mask)
+    )
+    (pad 32 smd rect (at 4.3 -0.75) (size 1.4 0.3)
+      (layers F.Cu F.Paste F.Mask)
+    )
+    (pad 33 smd rect (at 4.3 -1.25) (size 1.4 0.3)
+      (layers F.Cu F.Paste F.Mask)
+    )
+    (pad 34 smd rect (at 4.3 -1.75) (size 1.4 0.3)
+      (layers F.Cu F.Paste F.Mask)
+    )
+    (pad 35 smd rect (at 4.3 -2.25) (size 1.4 0.3)
+      (layers F.Cu F.Paste F.Mask)
+    )
+    (pad 36 smd rect (at 4.3 -2.75) (size 1.4 0.3)
+      (layers F.Cu F.Paste F.Mask)
+    )
+    (pad 37 smd rect (at 2.75 -4.3) (size 0.3 1.4)
+      (layers F.Cu F.Paste F.Mask)
+    )
+    (pad 38 smd rect (at 2.25 -4.3) (size 0.3 1.4)
+      (layers F.Cu F.Paste F.Mask)
+    )
+    (pad 39 smd rect (at 1.75 -4.3) (size 0.3 1.4)
+      (layers F.Cu F.Paste F.Mask)
+    )
+    (pad 40 smd rect (at 1.25 -4.3) (size 0.3 1.4)
+      (layers F.Cu F.Paste F.Mask)
+    )
+    (pad 41 smd rect (at 0.75 -4.3) (size 0.3 1.4)
+      (layers F.Cu F.Paste F.Mask)
+    )
+    (pad 42 smd rect (at 0.25 -4.3) (size 0.3 1.4)
+      (layers F.Cu F.Paste F.Mask)
+    )
+    (pad 43 smd rect (at -0.25 -4.3) (size 0.3 1.4)
+      (layers F.Cu F.Paste F.Mask)
+    )
+    (pad 44 smd rect (at -0.75 -4.3) (size 0.3 1.4)
+      (layers F.Cu F.Paste F.Mask)
+    )
+    (pad 45 smd rect (at -1.25 -4.3) (size 0.3 1.4)
+      (layers F.Cu F.Paste F.Mask)
+    )
+    (pad 46 smd rect (at -1.75 -4.3) (size 0.3 1.4)
+      (layers F.Cu F.Paste F.Mask)
+    )
+    (pad 47 smd rect (at -2.25 -4.3) (size 0.3 1.4)
+      (layers F.Cu F.Paste F.Mask)
+    )
+    (pad 48 smd rect (at -2.75 -4.3) (size 0.3 1.4)
+      (layers F.Cu F.Paste F.Mask)
+    )
+    (model ../3d_models/ab2_lqfp/AB2_LQFP48.wrl
+      (at (xyz 0 0 0))
+      (scale (xyz 0.3937 0.3937 0.3937))
+      (rotate (xyz 0 0 -90))
+    )
+  )

Commit message: AB2-K03D: add lqfp 60 pin render problems
Parts:
- removed AB2_0805_C_125: VAL**, AB2_0805_C_125
- removed AB2_0805_C_60: VAL**, AB2_0805_C_60
- removed AB2_0805_C_80: VAL**, AB2_0805_C_80
- removed AB2_LQFP48: VAL**, AB2_LQFP48
Changed lines of the file:
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@@
     (links 0)
     (no_connects 0)
-    (area 7.723012 12.0015 151.447501 284.669892)
+    (area 7.723012 12.0015 151.447501 233.743501)
     (thickness 1.6)
     (drawings 0)
     (tracks 0)
     (zones 0)
-    (modules 104)
+    (modules 100)
     (nets 6)
   )
@@
     (mod_text_size 1 1)
     (mod_text_width 0.15)
-    (pad_size 1.6764 1.6764)
-    (pad_drill 1.016)
+    (pad_size 1.4 0.3)
+    (pad_drill 0)
     (pad_to_mask_clearance 0)
     (aux_axis_origin 199.898 142.494)
@@
     )
   )
-  (module AB2_0805_C_60 (layer F.Cu)
-    (at 76.2 15.24)
-    (fp_text reference AB2_0805_C_60 (at 0 -1.27) (layer F.SilkS)
-      (effects (font (size 0.8128 0.8128) (thickness 0.0762)))
-    )
-    (fp_text value VAL** (at 0 1.27) (layer F.SilkS)
-      (effects (font (size 0.8128 0.8128) (thickness 0.0762)))
-    )
-    (fp_line (start -0.29972 0.59944) (end 0.29972 0.59944) (layer F.SilkS) (width 0.127))
-    (fp_line (start -0.29972 -0.59944) (end 0.29972 -0.59944) (layer F.SilkS) (width 0.127))
-    (pad 1 smd rect (at -0.9 0) (size 0.8 1.2)
-      (layers F.Cu F.Paste F.Mask)
-    )
-    (pad 2 smd rect (at 0.9 0) (size 0.8 1.2)
-      (layers F.Cu F.Paste F.Mask)
-    )
-    (model "../../../../Program Files (x86)/KiCad/share/3d_models/ab2_passive/AB2_0805_C_60.wrl"
-      (at (xyz 0 0 0))
-      (scale (xyz 0.3937 0.3937 0.3937))
-      (rotate (xyz 0 0 0))
-    )
-  )
-  (module AB2_0805_C_80 (layer F.Cu)
-    (at 76.2 17.78)
-    (fp_text reference AB2_0805_C_80 (at 0 -1.27) (layer F.SilkS)
-      (effects (font (size 0.8128 0.8128) (thickness 0.0762)))
-    )
-    (fp_text value VAL** (at 0 1.27) (layer F.SilkS)
-      (effects (font (size 0.8128 0.8128) (thickness 0.0762)))
-    )
-    (fp_line (start -0.29972 0.59944) (end 0.29972 0.59944) (layer F.SilkS) (width 0.127))
-    (fp_line (start -0.29972 -0.59944) (end 0.29972 -0.59944) (layer F.SilkS) (width 0.127))
-    (pad 1 smd rect (at -0.9 0) (size 0.8 1.2)
-      (layers F.Cu F.Paste F.Mask)
-    )
-    (pad 2 smd rect (at 0.9 0) (size 0.8 1.2)
-      (layers F.Cu F.Paste F.Mask)
-    )
-    (model "../../../../Program Files (x86)/KiCad/share/3d_models/ab2_passive/AB2_0805_C_80.wrl"
-      (at (xyz 0 0 0))
-      (scale (xyz 0.3937 0.3937 0.3937))
-      (rotate (xyz 0 0 0))
-    )
-  )
-  (module AB2_0805_C_125 (layer F.Cu)
-    (at 76.2 20.32)
-    (fp_text reference AB2_0805_C_125 (at 0 -1.27) (layer F.SilkS)
-      (effects (font (size 0.8128 0.8128) (thickness 0.0762)))
-    )
-    (fp_text value VAL** (at 0 1.27) (layer F.SilkS)
-      (effects (font (size 0.8128 0.8128) (thickness 0.0762)))
-    )
-    (fp_line (start -0.29972 0.59944) (end 0.29972 0.59944) (layer F.SilkS) (width 0.127))
-    (fp_line (start -0.29972 -0.59944) (end 0.29972 -0.59944) (layer F.SilkS) (width 0.127))
-    (pad 1 smd rect (at -0.9 0) (size 0.8 1.2)
-      (layers F.Cu F.Paste F.Mask)
-    )
-    (pad 2 smd rect (at 0.9 0) (size 0.8 1.2)
-      (layers F.Cu F.Paste F.Mask)
-    )
-    (model "../../../../Program Files (x86)/KiCad/share/3d_models/ab2_passive/AB2_0805_C_125.wrl"
-      (at (xyz 0 0 0))
-      (scale (xyz 0.3937 0.3937 0.3937))
-      (rotate (xyz 0 0 0))
-    )
-  )
-  (module AB2_LQFP48 (layer F.Cu)
-    (at 17.78 279.4)
-    (fp_text reference AB2_LQFP48 (at 0 -1.27) (layer F.SilkS)
-      (effects (font (size 0.8128 0.8128) (thickness 0.0762)))
-    )
-    (fp_text value VAL** (at 0 1.27) (layer F.SilkS)
-      (effects (font (size 0.8128 0.8128) (thickness 0.0762)))
-    )
-    (fp_circle (center -2.8 -2.8) (end -2.8 -3.1) (layer F.SilkS) (width 0.127))
-    (fp_line (start -3.5 -3.5) (end 3.5 -3.5) (layer F.SilkS) (width 0.127))
-    (fp_line (start 3.5 -3.5) (end 3.5 3.5) (layer F.SilkS) (width 0.127))
-    (fp_line (start 3.5 3.5) (end -3.5 3.5) (layer F.SilkS) (width 0.127))
-    (fp_line (start -3.5 3.5) (end -3.5 -3.5) (layer F.SilkS) (width 0.127))
-    (pad 6 smd rect (at -4.3 -0.25) (size 1.4 0.3)
-      (layers F.Cu F.Paste F.Mask)
-    )
-    (pad 5 smd rect (at -4.3 -0.75) (size 1.4 0.3)
-      (layers F.Cu F.Paste F.Mask)
-    )
-    (pad 4 smd rect (at -4.3 -1.25) (size 1.4 0.3)
-      (layers F.Cu F.Paste F.Mask)
-    )
-    (pad 3 smd rect (at -4.3 -1.75) (size 1.4 0.3)
-      (layers F.Cu F.Paste F.Mask)
-    )
-    (pad 2 smd rect (at -4.3 -2.25) (size 1.4 0.3)
-      (layers F.Cu F.Paste F.Mask)
-    )
-    (pad 1 smd rect (at -4.3 -2.75) (size 1.4 0.3)
-      (layers F.Cu F.Paste F.Mask)
-    )
-    (pad 7 smd rect (at -4.3 0.25) (size 1.4 0.3)
-      (layers F.Cu F.Paste F.Mask)
-    )
-    (pad 8 smd rect (at -4.3 0.75) (size 1.4 0.3)
-      (layers F.Cu F.Paste F.Mask)
-    )
-    (pad 9 smd rect (at -4.3 1.25) (size 1.4 0.3)
-      (layers F.Cu F.Paste F.Mask)
-    )
-    (pad 10 smd rect (at -4.3 1.75) (size 1.4 0.3)
-      (layers F.Cu F.Paste F.Mask)
-    )
-    (pad 11 smd rect (at -4.3 2.25) (size 1.4 0.3)
-      (layers F.Cu F.Paste F.Mask)
-    )
-    (pad 12 smd rect (at -4.3 2.75) (size 1.4 0.3)
-      (layers F.Cu F.Paste F.Mask)
-    )
-    (pad 13 smd rect (at -2.75 4.3) (size 0.3 1.4)
-      (layers F.Cu F.Paste F.Mask)
-    )
-    (pad 14 smd rect (at -2.25 4.3) (size 0.3 1.4)
-      (layers F.Cu F.Paste F.Mask)
-    )
-    (pad 15 smd rect (at -1.75 4.3) (size 0.3 1.4)
-      (layers F.Cu F.Paste F.Mask)
-    )
-    (pad 16 smd rect (at -1.25 4.3) (size 0.3 1.4)
-      (layers F.Cu F.Paste F.Mask)
-    )
-    (pad 17 smd rect (at -0.75 4.3) (size 0.3 1.4)
-      (layers F.Cu F.Paste F.Mask)
-    )
-    (pad 18 smd rect (at -0.25 4.3) (size 0.3 1.4)
-      (layers F.Cu F.Paste F.Mask)
-    )
-    (pad 19 smd rect (at 0.25 4.3) (size 0.3 1.4)
-      (layers F.Cu F.Paste F.Mask)
-    )
-    (pad 20 smd rect (at 0.75 4.3) (size 0.3 1.4)
-      (layers F.Cu F.Paste F.Mask)
-    )
-    (pad 21 smd rect (at 1.25 4.3) (size 0.3 1.4)
-      (layers F.Cu F.Paste F.Mask)
-    )
-    (pad 22 smd rect (at 1.75 4.3) (size 0.3 1.4)
-      (layers F.Cu F.Paste F.Mask)
-    )
-    (pad 23 smd rect (at 2.25 4.3) (size 0.3 1.4)
-      (layers F.Cu F.Paste F.Mask)
-    )
-    (pad 24 smd rect (at 2.75 4.3) (size 0.3 1.4)
-      (layers F.Cu F.Paste F.Mask)
-    )
-    (pad 25 smd rect (at 4.3 2.75) (size 1.4 0.3)
-      (layers F.Cu F.Paste F.Mask)
-    )
-    (pad 26 smd rect (at 4.3 2.25) (size 1.4 0.3)
-      (layers F.Cu F.Paste F.Mask)
-    )
-    (pad 27 smd rect (at 4.3 1.75) (size 1.4 0.3)
-      (layers F.Cu F.Paste F.Mask)
-    )
-    (pad 28 smd rect (at 4.3 1.25) (size 1.4 0.3)
-      (layers F.Cu F.Paste F.Mask)
-    )
-    (pad 29 smd rect (at 4.3 0.75) (size 1.4 0.3)
-      (layers F.Cu F.Paste F.Mask)
-    )
-    (pad 30 smd rect (at 4.3 0.25) (size 1.4 0.3)
-      (layers F.Cu F.Paste F.Mask)
-    )
-    (pad 31 smd rect (at 4.3 -0.25) (size 1.4 0.3)
-      (layers F.Cu F.Paste F.Mask)
-    )
-    (pad 32 smd rect (at 4.3 -0.75) (size 1.4 0.3)
-      (layers F.Cu F.Paste F.Mask)
-    )
-    (pad 33 smd rect (at 4.3 -1.25) (size 1.4 0.3)
-      (layers F.Cu F.Paste F.Mask)
-    )
-    (pad 34 smd rect (at 4.3 -1.75) (size 1.4 0.3)
-      (layers F.Cu F.Paste F.Mask)
-    )
-    (pad 35 smd rect (at 4.3 -2.25) (size 1.4 0.3)
-      (layers F.Cu F.Paste F.Mask)
-    )
-    (pad 36 smd rect (at 4.3 -2.75) (size 1.4 0.3)
-      (layers F.Cu F.Paste F.Mask)
-    )
-    (pad 37 smd rect (at 2.75 -4.3) (size 0.3 1.4)
-      (layers F.Cu F.Paste F.Mask)
-    )
-    (pad 38 smd rect (at 2.25 -4.3) (size 0.3 1.4)
-      (layers F.Cu F.Paste F.Mask)
-    )
-    (pad 39 smd rect (at 1.75 -4.3) (size 0.3 1.4)
-      (layers F.Cu F.Paste F.Mask)
-    )
-    (pad 40 smd rect (at 1.25 -4.3) (size 0.3 1.4)
-      (layers F.Cu F.Paste F.Mask)
-    )
-    (pad 41 smd rect (at 0.75 -4.3) (size 0.3 1.4)
-      (layers F.Cu F.Paste F.Mask)
-    )
-    (pad 42 smd rect (at 0.25 -4.3) (size 0.3 1.4)
-      (layers F.Cu F.Paste F.Mask)
-    )
-    (pad 43 smd rect (at -0.25 -4.3) (size 0.3 1.4)
-      (layers F.Cu F.Paste F.Mask)
-    )
-    (pad 44 smd rect (at -0.75 -4.3) (size 0.3 1.4)
-      (layers F.Cu F.Paste F.Mask)
-    )
-    (pad 45 smd rect (at -1.25 -4.3) (size 0.3 1.4)
-      (layers F.Cu F.Paste F.Mask)
-    )
-    (pad 46 smd rect (at -1.75 -4.3) (size 0.3 1.4)
-      (layers F.Cu F.Paste F.Mask)
-    )
-    (pad 47 smd rect (at -2.25 -4.3) (size 0.3 1.4)
-      (layers F.Cu F.Paste F.Mask)
-    )
-    (pad 48 smd rect (at -2.75 -4.3) (size 0.3 1.4)
-      (layers F.Cu F.Paste F.Mask)
-    )
-    (model ../3d_models/ab2_lqfp/AB2_LQFP48.wrl
-      (at (xyz 0 0 0))
-      (scale (xyz 0.3937 0.3937 0.3937))
-      (rotate (xyz 0 0 -90))
-    )
-  )
