File: 3d_models/AB2-K03D - Demo/AB2-K03D - Demo_master.kicad_pcb (KiCad board)
At the start: 2 copper layers, 222 parts

Commit message: 3d_models: AB2-K03D: add 2x5 shrouded hdr to main
Parts:
- added AB2_HDR_M05-2V: VAL**, AB2_HDR_M05-2V-S, F.Cu at (204.5, 161.3)
Changed lines of the file:
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@@
     (tracks 0)
     (zones 0)
-    (modules 222)
+    (modules 223)
     (nets 1)
   )
@@
     )
   )
+  (module AB2_HDR_M05-2V-S (layer F.Cu)
+    (at 204.47 161.29)
+    (fp_text reference AB2_HDR_M05-2V (at 0 5.08) (layer F.SilkS)
+      (effects (font (size 0.8128 0.8128) (thickness 0.0762)))
+    )
+    (fp_text value VAL** (at 0 -5.08) (layer F.SilkS)
+      (effects (font (size 0.8128 0.8128) (thickness 0.0762)))
+    )
+    (fp_line (start 2.032 3.302) (end 2.032 4.191) (layer F.SilkS) (width 0.127))
+    (fp_line (start -2.032 3.302) (end -2.032 4.191) (layer F.SilkS) (width 0.127))
+    (fp_line (start -4.953 2.794) (end -5.08 2.921) (layer F.SilkS) (width 0.127))
+    (fp_line (start -5.207 2.794) (end -5.08 2.921) (layer F.SilkS) (width 0.127))
+    (fp_line (start -5.334 2.794) (end -5.08 3.048) (layer F.SilkS) (width 0.127))
+    (fp_line (start -5.08 3.048) (end -4.826 2.794) (layer F.SilkS) (width 0.127))
+    (fp_line (start -4.826 2.794) (end -5.334 2.794) (layer F.SilkS) (width 0.127))
+    (fp_line (start 9.017 -3.302) (end -9.017 -3.302) (layer F.SilkS) (width 0.127))
+    (fp_line (start -9.017 -3.302) (end -9.017 3.302) (layer F.SilkS) (width 0.127))
+    (fp_line (start -9.017 3.302) (end 9.017 3.302) (layer F.SilkS) (width 0.127))
+    (fp_line (start 9.017 3.302) (end 9.017 -3.302) (layer F.SilkS) (width 0.127))
+    (fp_line (start 10.16 -4.191) (end -10.16 -4.191) (layer F.SilkS) (width 0.127))
+    (fp_line (start -10.16 -4.191) (end -10.16 4.191) (layer F.SilkS) (width 0.127))
+    (fp_line (start -10.16 4.191) (end 10.16 4.191) (layer F.SilkS) (width 0.127))
+    (fp_line (start 10.16 4.191) (end 10.16 -4.191) (layer F.SilkS) (width 0.127))
+    (fp_line (start 3.81 -1.905) (end 4.445 -2.54) (layer F.SilkS) (width 0.127))
+    (fp_line (start 4.445 -2.54) (end 5.715 -2.54) (layer F.SilkS) (width 0.127))
+    (fp_line (start 5.715 -2.54) (end 6.35 -1.905) (layer F.SilkS) (width 0.127))
+    (fp_line (start 6.35 -1.905) (end 6.35 1.905) (layer F.SilkS) (width 0.127))
+    (fp_line (start 6.35 1.905) (end 5.715 2.54) (layer F.SilkS) (width 0.127))
+    (fp_line (start 5.715 2.54) (end 4.445 2.54) (layer F.SilkS) (width 0.127))
+    (fp_line (start 4.445 2.54) (end 3.81 1.905) (layer F.SilkS) (width 0.127))
+    (fp_line (start 1.27 -1.905) (end 1.905 -2.54) (layer F.SilkS) (width 0.127))
+    (fp_line (start 1.905 -2.54) (end 3.175 -2.54) (layer F.SilkS) (width 0.127))
+    (fp_line (start 3.175 -2.54) (end 3.81 -1.905) (layer F.SilkS) (width 0.127))
+    (fp_line (start 3.81 -1.905) (end 3.81 1.905) (layer F.SilkS) (width 0.127))
+    (fp_line (start 3.81 1.905) (end 3.175 2.54) (layer F.SilkS) (width 0.127))
+    (fp_line (start 3.175 2.54) (end 1.905 2.54) (layer F.SilkS) (width 0.127))
+    (fp_line (start 1.905 2.54) (end 1.27 1.905) (layer F.SilkS) (width 0.127))
+    (fp_line (start -1.27 -1.905) (end -0.635 -2.54) (layer F.SilkS) (width 0.127))
+    (fp_line (start -0.635 -2.54) (end 0.635 -2.54) (layer F.SilkS) (width 0.127))
+    (fp_line (start 0.635 -2.54) (end 1.27 -1.905) (layer F.SilkS) (width 0.127))
+    (fp_line (start 1.27 -1.905) (end 1.27 1.905) (layer F.SilkS) (width 0.127))
+    (fp_line (start 1.27 1.905) (end 0.635 2.54) (layer F.SilkS) (width 0.127))
+    (fp_line (start 0.635 2.54) (end -0.635 2.54) (layer F.SilkS) (width 0.127))
+    (fp_line (start -0.635 2.54) (end -1.27 1.905) (layer F.SilkS) (width 0.127))
+    (fp_line (start -3.81 -1.905) (end -3.175 -2.54) (layer F.SilkS) (width 0.127))
+    (fp_line (start -3.175 -2.54) (end -1.905 -2.54) (layer F.SilkS) (width 0.127))
+    (fp_line (start -1.905 -2.54) (end -1.27 -1.905) (layer F.SilkS) (width 0.127))
+    (fp_line (start -1.27 -1.905) (end -1.27 1.905) (layer F.SilkS) (width 0.127))
+    (fp_line (start -1.27 1.905) (end -1.905 2.54) (layer F.SilkS) (width 0.127))
+    (fp_line (start -1.905 2.54) (end -3.175 2.54) (layer F.SilkS) (width 0.127))
+    (fp_line (start -3.175 2.54) (end -3.81 1.905) (layer F.SilkS) (width 0.127))
+    (fp_line (start -5.715 2.54) (end -6.35 1.905) (layer F.SilkS) (width 0.127))
+    (fp_line (start -6.35 1.905) (end -6.35 -1.905) (layer F.SilkS) (width 0.127))
+    (fp_line (start -6.35 -1.905) (end -5.715 -2.54) (layer F.SilkS) (width 0.127))
+    (fp_line (start -5.715 -2.54) (end -4.445 -2.54) (layer F.SilkS) (width 0.127))
+    (fp_line (start -4.445 -2.54) (end -3.81 -1.905) (layer F.SilkS) (width 0.127))
+    (fp_line (start -3.81 -1.905) (end -3.81 1.905) (layer F.SilkS) (width 0.127))
+    (fp_line (start -3.81 1.905) (end -4.445 2.54) (layer F.SilkS) (width 0.127))
+    (fp_line (start -4.445 2.54) (end -5.715 2.54) (layer F.SilkS) (width 0.127))
+    (pad 1 thru_hole circle (at -5.08 1.27) (size 1.6764 1.6764) (drill 1.016)
+      (layers *.Cu *.Mask F.SilkS)
+    )
+    (pad 2 thru_hole circle (at -5.08 -1.27) (size 1.6764 1.6764) (drill 1.016)
+      (layers *.Cu *.Mask F.SilkS)
+    )
+    (pad 3 thru_hole circle (at -2.54 1.27) (size 1.6764 1.6764) (drill 1.016)
+      (layers *.Cu *.Mask F.SilkS)
+    )
+    (pad 4 thru_hole circle (at -2.54 -1.27) (size 1.6764 1.6764) (drill 1.016)
+      (layers *.Cu *.Mask F.SilkS)
+    )
+    (pad 5 thru_hole circle (at 0 1.27) (size 1.6764 1.6764) (drill 1.016)
+      (layers *.Cu *.Mask F.SilkS)
+    )
+    (pad 6 thru_hole circle (at 0 -1.27) (size 1.6764 1.6764) (drill 1.016)
+      (layers *.Cu *.Mask F.SilkS)
+    )
+    (pad 7 thru_hole circle (at 2.54 1.27) (size 1.6764 1.6764) (drill 1.016)
+      (layers *.Cu *.Mask F.SilkS)
+    )
+    (pad 8 thru_hole circle (at 2.54 -1.27) (size 1.6764 1.6764) (drill 1.016)
+      (layers *.Cu *.Mask F.SilkS)
+    )
+    (pad 9 thru_hole circle (at 5.08 1.27) (size 1.6764 1.6764) (drill 1.016)
+      (layers *.Cu *.Mask F.SilkS)
+    )
+    (pad 10 thru_hole circle (at 5.08 -1.27) (size 1.6764 1.6764) (drill 1.016)
+      (layers *.Cu *.Mask F.SilkS)
+    )
+    (model ../3d_models/ab2_idc/AB2_HDR_M05-2V-S-3M.wrl
+      (at (xyz 0 0 0))
+      (scale (xyz 0.3937 0.3937 0.3937))
+      (rotate (xyz 0 0 0))
+    )
+  )
