File: 3d_models/AB2-K03D - Demo/AB2-K03D - Demo_ic_packages.kicad_pcb (KiCad board)
At the start: 2 copper layers, 27 parts

Commit message: 3d: AB2-K03D: ic_pckgs: update all
Parts:
- removed AB2_TSSOP30: VAL**, AB2_TSSOP30
- removed AB2_TSSOP32: VAL**, AB2_TSSOP32
- added AB2_TSSOP28_0p50P: VAL**, AB2_TSSOP28_0p50P, F.Cu at (83.8, 177.8)
- added AB2_TSSOP30_0p50P: VAL**, AB2_TSSOP30_0p50P, F.Cu at (106.7, 177.8)
- added AB2_TSSOP30_W: VAL**, AB2_TSSOP30_W, F.Cu at (95.2, 177.8)
- added AB2_TSSOP32_W: VAL**, AB2_TSSOP32_W, F.Cu at (118.1, 177.8)
- added AB2_TSSOP38_0p50P: VAL**, AB2_TSSOP38_0p50P, F.Cu at (185.4, 177.8)
- added AB2_TSSOP38_PWP: VAL**, AB2_TSSOP38_PWP, F.Cu at (144.8, 177.8)
- added AB2_TSSOP38_PWP_0p50P: VAL**, AB2_TSSOP38_PWP_0p50P, F.Cu at (196.8, 177.8)
- added AB2_TSSOP38_PWP_SLUG: VAL**, AB2_TSSOP38_PWP_SLUG, F.Cu at (158.8, 177.8)
- added AB2_TSSOP38_PWP_SLUG_0p50P: VAL**, AB2_TSSOP38_PWP_SLUG_0p50P, F.Cu at (208.3, 177.8)
- added AB2_TSSOP38_W: VAL**, AB2_TSSOP38_W, F.Cu at (172.7, 177.8)
- AB2_TSSOP44_0p50P: renamed from AB2_TSSOP44; footprint AB2_TSSOP44 -> AB2_TSSOP44_0p50P
- AB2_TSSOP50_0p50P: renamed from AB2_TSSOP50; footprint AB2_TSSOP50 -> AB2_TSSOP50_0p50P
- moved AB2_TSSOP44_0p50P 92.7 mm to (219.7, 177.8)
- moved AB2_TSSOP50_0p50P 91.4 mm to (232.4, 177.8)
- moved AB2_TSSOP38 17.8 mm to (130.8, 177.8)
