File: 3d_models/AB2-K03D - Demo/AB2-K03D - Demo_headers.kicad_pcb (KiCad board)
At the start: 2 copper layers, 125 parts

Commit message: 3d_models: AB2-K03D: add 2x3 and 2x4 shroud hdrs
Parts:
- added AB2_HDR_M03-2V-S: VAL**, AB2_HDR_M03-2V-S, F.Cu at (21.6, 279.4)
- added AB2_HDR_M04-2V-S: VAL**, AB2_HDR_M04-2V-S, F.Cu at (22.9, 268.0)
Changed lines of the file:
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@@
     (links 0)
     (no_connects 0)
-    (area 8.1915 110.593012 302.9585 286.4485)
+    (area 7.356123 3.746499 286.067501 207.7085)
     (thickness 1.6)
     (drawings 0)
     (tracks 0)
     (zones 0)
-    (modules 125)
+    (modules 127)
     (nets 1)
   )
@@
       (scale (xyz 0.3937 0.3937 0.3937))
       (rotate (xyz 0 0 0))
+    )
+  )
+  (module AB2_HDR_M03-2V-S (layer F.Cu)
+    (at 21.59 279.4)
+    (fp_text reference AB2_HDR_M03-2V-S (at 0 5.08) (layer F.SilkS)
+      (effects (font (size 0.8128 0.8128) (thickness 0.0762)))
+    )
+    (fp_text value VAL** (at 0 -5.08) (layer F.SilkS)
+      (effects (font (size 0.8128 0.8128) (thickness 0.0762)))
+    )
+    (fp_line (start 2.032 3.302) (end 2.032 4.191) (layer F.SilkS) (width 0.127))
+    (fp_line (start -2.032 3.302) (end -2.032 4.191) (layer F.SilkS) (width 0.127))
+    (fp_line (start -2.794 2.794) (end -2.286 2.794) (layer F.SilkS) (width 0.127))
+    (fp_line (start -2.413 2.794) (end -2.54 2.921) (layer F.SilkS) (width 0.127))
+    (fp_line (start -2.667 2.794) (end -2.54 2.921) (layer F.SilkS) (width 0.127))
+    (fp_line (start -2.286 2.794) (end -2.54 3.048) (layer F.SilkS) (width 0.127))
+    (fp_line (start -2.794 2.794) (end -2.54 3.048) (layer F.SilkS) (width 0.127))
+    (fp_line (start 6.477 -3.302) (end -6.477 -3.302) (layer F.SilkS) (width 0.127))
+    (fp_line (start -6.477 -3.302) (end -6.477 3.302) (layer F.SilkS) (width 0.127))
+    (fp_line (start -6.477 3.302) (end 6.477 3.302) (layer F.SilkS) (width 0.127))
+    (fp_line (start 6.477 3.302) (end 6.477 -3.302) (layer F.SilkS) (width 0.127))
+    (fp_line (start 7.62 -4.191) (end -7.62 -4.191) (layer F.SilkS) (width 0.127))
+    (fp_line (start -7.62 -4.191) (end -7.62 4.191) (layer F.SilkS) (width 0.127))
+    (fp_line (start -7.62 4.191) (end 7.62 4.191) (layer F.SilkS) (width 0.127))
+    (fp_line (start 7.62 4.191) (end 7.62 -4.191) (layer F.SilkS) (width 0.127))
+    (fp_line (start -2.794 2.54) (end -2.286 2.54) (layer F.SilkS) (width 0.127))
+    (fp_line (start 1.27 -1.905) (end 1.905 -2.54) (layer F.SilkS) (width 0.127))
+    (fp_line (start 1.905 -2.54) (end 3.175 -2.54) (layer F.SilkS) (width 0.127))
+    (fp_line (start 3.175 -2.54) (end 3.81 -1.905) (layer F.SilkS) (width 0.127))
+    (fp_line (start 3.81 -1.905) (end 3.81 1.905) (layer F.SilkS) (width 0.127))
+    (fp_line (start 3.81 1.905) (end 3.175 2.54) (layer F.SilkS) (width 0.127))
+    (fp_line (start 3.175 2.54) (end 1.905 2.54) (layer F.SilkS) (width 0.127))
+    (fp_line (start 1.905 2.54) (end 1.27 1.905) (layer F.SilkS) (width 0.127))
+    (fp_line (start -1.27 -1.905) (end -0.635 -2.54) (layer F.SilkS) (width 0.127))
+    (fp_line (start -0.635 -2.54) (end 0.635 -2.54) (layer F.SilkS) (width 0.127))
+    (fp_line (start 0.635 -2.54) (end 1.27 -1.905) (layer F.SilkS) (width 0.127))
+    (fp_line (start 1.27 -1.905) (end 1.27 1.905) (layer F.SilkS) (width 0.127))
+    (fp_line (start 1.27 1.905) (end 0.635 2.54) (layer F.SilkS) (width 0.127))
+    (fp_line (start 0.635 2.54) (end -0.635 2.54) (layer F.SilkS) (width 0.127))
+    (fp_line (start -0.635 2.54) (end -1.27 1.905) (layer F.SilkS) (width 0.127))
+    (fp_line (start -3.175 2.54) (end -3.81 1.905) (layer F.SilkS) (width 0.127))
+    (fp_line (start -3.81 1.905) (end -3.81 -1.905) (layer F.SilkS) (width 0.127))
+    (fp_line (start -3.81 -1.905) (end -3.175 -2.54) (layer F.SilkS) (width 0.127))
+    (fp_line (start -3.175 -2.54) (end -1.905 -2.54) (layer F.SilkS) (width 0.127))
+    (fp_line (start -1.905 -2.54) (end -1.27 -1.905) (layer F.SilkS) (width 0.127))
+    (fp_line (start -1.27 -1.905) (end -1.27 1.905) (layer F.SilkS) (width 0.127))
+    (fp_line (start -1.27 1.905) (end -1.905 2.54) (layer F.SilkS) (width 0.127))
+    (fp_line (start -1.905 2.54) (end -3.175 2.54) (layer F.SilkS) (width 0.127))
+    (pad 1 thru_hole circle (at -2.54 1.27) (size 1.6764 1.6764) (drill 1.016)
+      (layers *.Cu *.Mask F.SilkS)
+    )
+    (pad 2 thru_hole circle (at -2.54 -1.27) (size 1.6764 1.6764) (drill 1.016)
+      (layers *.Cu *.Mask F.SilkS)
+    )
+    (pad 3 thru_hole circle (at 0 1.27) (size 1.6764 1.6764) (drill 1.016)
+      (layers *.Cu *.Mask F.SilkS)
+    )
+    (pad 4 thru_hole circle (at 0 -1.27) (size 1.6764 1.6764) (drill 1.016)
+      (layers *.Cu *.Mask F.SilkS)
+    )
+    (pad 5 thru_hole circle (at 2.54 1.27) (size 1.6764 1.6764) (drill 1.016)
+      (layers *.Cu *.Mask F.SilkS)
+    )
+    (pad 6 thru_hole circle (at 2.54 -1.27) (size 1.6764 1.6764) (drill 1.016)
+      (layers *.Cu *.Mask F.SilkS)
+    )
+    (model ../3d_models/ab2_idc/AB2_HDR_M03-2V-S-3M.wrl
+      (at (xyz 0 0 0))
+      (scale (xyz 0.3937 0.3937 0.3937))
+      (rotate (xyz 0 0 0))
+    )
+  )
+  (module AB2_HDR_M04-2V-S (layer F.Cu)
+    (at 22.86 267.97)
+    (path AB2_HDR05_2)
+    (fp_text reference AB2_HDR_M04-2V-S (at 0 5.08) (layer F.SilkS)
+      (effects (font (size 0.8128 0.8128) (thickness 0.0762)))
+    )
+    (fp_text value VAL** (at 0 -5.08) (layer F.SilkS)
+      (effects (font (size 0.8128 0.8128) (thickness 0.0762)))
+    )
+    (fp_line (start 2.032 3.302) (end 2.032 4.191) (layer F.SilkS) (width 0.127))
+    (fp_line (start -2.032 3.302) (end -2.032 4.191) (layer F.SilkS) (width 0.127))
+    (fp_line (start 7.747 -3.302) (end -7.747 -3.302) (layer F.SilkS) (width 0.127))
+    (fp_line (start -7.747 -3.302) (end -7.747 3.302) (layer F.SilkS) (width 0.127))
+    (fp_line (start -7.747 3.302) (end 7.747 3.302) (layer F.SilkS) (width 0.127))
+    (fp_line (start 7.747 3.302) (end 7.747 -3.302) (layer F.SilkS) (width 0.127))
+    (fp_line (start 8.89 -4.191) (end -8.89 -4.191) (layer F.SilkS) (width 0.127))
+    (fp_line (start -8.89 -4.191) (end -8.89 4.191) (layer F.SilkS) (width 0.127))
+    (fp_line (start -8.89 4.191) (end 8.89 4.191) (layer F.SilkS) (width 0.127))
+    (fp_line (start 8.89 4.191) (end 8.89 -4.191) (layer F.SilkS) (width 0.127))
+    (fp_line (start -4.064 2.794) (end -3.556 2.794) (layer F.SilkS) (width 0.127))
+    (fp_line (start -3.683 2.794) (end -3.81 2.921) (layer F.SilkS) (width 0.127))
+    (fp_line (start -3.937 2.794) (end -3.81 2.921) (layer F.SilkS) (width 0.127))
+    (fp_line (start -3.556 2.794) (end -3.81 3.048) (layer F.SilkS) (width 0.127))
+    (fp_line (start -4.064 2.794) (end -3.81 3.048) (layer F.SilkS) (width 0.127))
+    (fp_line (start 2.54 -1.905) (end 3.175 -2.54) (layer F.SilkS) (width 0.127))
+    (fp_line (start 3.175 -2.54) (end 4.445 -2.54) (layer F.SilkS) (width 0.127))
+    (fp_line (start 4.445 -2.54) (end 5.08 -1.905) (layer F.SilkS) (width 0.127))
+    (fp_line (start 5.08 -1.905) (end 5.08 1.905) (layer F.SilkS) (width 0.127))
+    (fp_line (start 5.08 1.905) (end 4.445 2.54) (layer F.SilkS) (width 0.127))
+    (fp_line (start 4.445 2.54) (end 3.175 2.54) (layer F.SilkS) (width 0.127))
+    (fp_line (start 3.175 2.54) (end 2.54 1.905) (layer F.SilkS) (width 0.127))
+    (fp_line (start 0 -1.905) (end 0.635 -2.54) (layer F.SilkS) (width 0.127))
+    (fp_line (start 0.635 -2.54) (end 1.905 -2.54) (layer F.SilkS) (width 0.127))
+    (fp_line (start 1.905 -2.54) (end 2.54 -1.905) (layer F.SilkS) (width 0.127))
+    (fp_line (start 2.54 -1.905) (end 2.54 1.905) (layer F.SilkS) (width 0.127))
+    (fp_line (start 2.54 1.905) (end 1.905 2.54) (layer F.SilkS) (width 0.127))
+    (fp_line (start 1.905 2.54) (end 0.635 2.54) (layer F.SilkS) (width 0.127))
+    (fp_line (start 0.635 2.54) (end 0 1.905) (layer F.SilkS) (width 0.127))
+    (fp_line (start -2.54 -1.905) (end -1.905 -2.54) (layer F.SilkS) (width 0.127))
+    (fp_line (start -1.905 -2.54) (end -0.635 -2.54) (layer F.SilkS) (width 0.127))
+    (fp_line (start -0.635 -2.54) (end 0 -1.905) (layer F.SilkS) (width 0.127))
+    (fp_line (start 0 -1.905) (end 0 1.905) (layer F.SilkS) (width 0.127))
+    (fp_line (start 0 1.905) (end -0.635 2.54) (layer F.SilkS) (width 0.127))
+    (fp_line (start -0.635 2.54) (end -1.905 2.54) (layer F.SilkS) (width 0.127))
+    (fp_line (start -1.905 2.54) (end -2.54 1.905) (layer F.SilkS) (width 0.127))
+    (fp_line (start -4.445 2.54) (end -5.08 1.905) (layer F.SilkS) (width 0.127))
+    (fp_line (start -5.08 1.905) (end -5.08 -1.905) (layer F.SilkS) (width 0.127))
+    (fp_line (start -5.08 -1.905) (end -4.445 -2.54) (layer F.SilkS) (width 0.127))
+    (fp_line (start -4.445 -2.54) (end -3.175 -2.54) (layer F.SilkS) (width 0.127))
+    (fp_line (start -3.175 -2.54) (end -2.54 -1.905) (layer F.SilkS) (width 0.127))
+    (fp_line (start -2.54 -1.905) (end -2.54 1.905) (layer F.SilkS) (width 0.127))
+    (fp_line (start -2.54 1.905) (end -3.175 2.54) (layer F.SilkS) (width 0.127))
+    (fp_line (start -3.175 2.54) (end -4.445 2.54) (layer F.SilkS) (width 0.127))
+    (pad 1 thru_hole circle (at -3.81 1.27) (size 1.6764 1.6764) (drill 1.016)
+      (layers *.Cu *.Mask F.SilkS)
+    )
+    (pad 2 thru_hole circle (at -3.81 -1.27) (size 1.6764 1.6764) (drill 1.016)
+      (layers *.Cu *.Mask F.SilkS)
+    )
+    (pad 3 thru_hole circle (at -1.27 1.27) (size 1.6764 1.6764) (drill 1.016)
+      (layers *.Cu *.Mask F.SilkS)
+    )
+    (pad 4 thru_hole circle (at -1.27 -1.27) (size 1.6764 1.6764) (drill 1.016)
+      (layers *.Cu *.Mask F.SilkS)
+    )
+    (pad 5 thru_hole circle (at 1.27 1.27) (size 1.6764 1.6764) (drill 1.016)
+      (layers *.Cu *.Mask F.SilkS)
+    )
+    (pad 6 thru_hole circle (at 1.27 -1.27) (size 1.6764 1.6764) (drill 1.016)
+      (layers *.Cu *.Mask F.SilkS)
+    )
+    (pad 7 thru_hole circle (at 3.81 1.27) (size 1.6764 1.6764) (drill 1.016)
+      (layers *.Cu *.Mask F.SilkS)
+    )
+    (pad 8 thru_hole circle (at 3.81 -1.27) (size 1.6764 1.6764) (drill 1.016)
+      (layers *.Cu *.Mask F.SilkS)
+    )
+    (model ../3d_models/ab2_idc/AB2_HDR_M04-2V-S-3M.wrl
+      (at (xyz 0 0 0))
+      (scale (xyz 0.3937 0.3937 0.3937))
+      (rotate (xyz 0 0 0))

Commit message: 3d_models: AB2-K03D: add 2x5 shrouded hdr
Parts:
- added AB2_HDR_M05-2V: VAL**, AB2_HDR_M05-2V-S, F.Cu at (24.1, 256.5)
Changed lines of the file:
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@@
     (links 0)
     (no_connects 0)
-    (area 7.356123 3.746499 286.067501 207.7085)
+    (area 7.356123 3.746499 286.067501 285.1785)
     (thickness 1.6)
     (drawings 0)
     (tracks 0)
     (zones 0)
-    (modules 127)
+    (modules 128)
     (nets 1)
   )
@@
       (at (xyz 0 0 0))
       (scale (xyz 0.3937 0.3937 0.3937))
+      (rotate (xyz 0 0 0))
+    )
+  )
+  (module AB2_HDR_M05-2V-S (layer F.Cu)
+    (at 24.13 256.54)
+    (fp_text reference AB2_HDR_M05-2V (at 0 5.08) (layer F.SilkS)
+      (effects (font (size 0.8128 0.8128) (thickness 0.0762)))
+    )
+    (fp_text value VAL** (at 0 -5.08) (layer F.SilkS)
+      (effects (font (size 0.8128 0.8128) (thickness 0.0762)))
+    )
+    (fp_line (start 2.032 3.302) (end 2.032 4.191) (layer F.SilkS) (width 0.127))
+    (fp_line (start -2.032 3.302) (end -2.032 4.191) (layer F.SilkS) (width 0.127))
+    (fp_line (start -4.953 2.794) (end -5.08 2.921) (layer F.SilkS) (width 0.127))
+    (fp_line (start -5.207 2.794) (end -5.08 2.921) (layer F.SilkS) (width 0.127))
+    (fp_line (start -5.334 2.794) (end -5.08 3.048) (layer F.SilkS) (width 0.127))
+    (fp_line (start -5.08 3.048) (end -4.826 2.794) (layer F.SilkS) (width 0.127))
+    (fp_line (start -4.826 2.794) (end -5.334 2.794) (layer F.SilkS) (width 0.127))
+    (fp_line (start 9.017 -3.302) (end -9.017 -3.302) (layer F.SilkS) (width 0.127))
+    (fp_line (start -9.017 -3.302) (end -9.017 3.302) (layer F.SilkS) (width 0.127))
+    (fp_line (start -9.017 3.302) (end 9.017 3.302) (layer F.SilkS) (width 0.127))
+    (fp_line (start 9.017 3.302) (end 9.017 -3.302) (layer F.SilkS) (width 0.127))
+    (fp_line (start 10.16 -4.191) (end -10.16 -4.191) (layer F.SilkS) (width 0.127))
+    (fp_line (start -10.16 -4.191) (end -10.16 4.191) (layer F.SilkS) (width 0.127))
+    (fp_line (start -10.16 4.191) (end 10.16 4.191) (layer F.SilkS) (width 0.127))
+    (fp_line (start 10.16 4.191) (end 10.16 -4.191) (layer F.SilkS) (width 0.127))
+    (fp_line (start 3.81 -1.905) (end 4.445 -2.54) (layer F.SilkS) (width 0.127))
+    (fp_line (start 4.445 -2.54) (end 5.715 -2.54) (layer F.SilkS) (width 0.127))
+    (fp_line (start 5.715 -2.54) (end 6.35 -1.905) (layer F.SilkS) (width 0.127))
+    (fp_line (start 6.35 -1.905) (end 6.35 1.905) (layer F.SilkS) (width 0.127))
+    (fp_line (start 6.35 1.905) (end 5.715 2.54) (layer F.SilkS) (width 0.127))
+    (fp_line (start 5.715 2.54) (end 4.445 2.54) (layer F.SilkS) (width 0.127))
+    (fp_line (start 4.445 2.54) (end 3.81 1.905) (layer F.SilkS) (width 0.127))
+    (fp_line (start 1.27 -1.905) (end 1.905 -2.54) (layer F.SilkS) (width 0.127))
+    (fp_line (start 1.905 -2.54) (end 3.175 -2.54) (layer F.SilkS) (width 0.127))
+    (fp_line (start 3.175 -2.54) (end 3.81 -1.905) (layer F.SilkS) (width 0.127))
+    (fp_line (start 3.81 -1.905) (end 3.81 1.905) (layer F.SilkS) (width 0.127))
+    (fp_line (start 3.81 1.905) (end 3.175 2.54) (layer F.SilkS) (width 0.127))
+    (fp_line (start 3.175 2.54) (end 1.905 2.54) (layer F.SilkS) (width 0.127))
+    (fp_line (start 1.905 2.54) (end 1.27 1.905) (layer F.SilkS) (width 0.127))
+    (fp_line (start -1.27 -1.905) (end -0.635 -2.54) (layer F.SilkS) (width 0.127))
+    (fp_line (start -0.635 -2.54) (end 0.635 -2.54) (layer F.SilkS) (width 0.127))
+    (fp_line (start 0.635 -2.54) (end 1.27 -1.905) (layer F.SilkS) (width 0.127))
+    (fp_line (start 1.27 -1.905) (end 1.27 1.905) (layer F.SilkS) (width 0.127))
+    (fp_line (start 1.27 1.905) (end 0.635 2.54) (layer F.SilkS) (width 0.127))
+    (fp_line (start 0.635 2.54) (end -0.635 2.54) (layer F.SilkS) (width 0.127))
+    (fp_line (start -0.635 2.54) (end -1.27 1.905) (layer F.SilkS) (width 0.127))
+    (fp_line (start -3.81 -1.905) (end -3.175 -2.54) (layer F.SilkS) (width 0.127))
+    (fp_line (start -3.175 -2.54) (end -1.905 -2.54) (layer F.SilkS) (width 0.127))
+    (fp_line (start -1.905 -2.54) (end -1.27 -1.905) (layer F.SilkS) (width 0.127))
+    (fp_line (start -1.27 -1.905) (end -1.27 1.905) (layer F.SilkS) (width 0.127))
+    (fp_line (start -1.27 1.905) (end -1.905 2.54) (layer F.SilkS) (width 0.127))
+    (fp_line (start -1.905 2.54) (end -3.175 2.54) (layer F.SilkS) (width 0.127))
+    (fp_line (start -3.175 2.54) (end -3.81 1.905) (layer F.SilkS) (width 0.127))
+    (fp_line (start -5.715 2.54) (end -6.35 1.905) (layer F.SilkS) (width 0.127))
+    (fp_line (start -6.35 1.905) (end -6.35 -1.905) (layer F.SilkS) (width 0.127))
+    (fp_line (start -6.35 -1.905) (end -5.715 -2.54) (layer F.SilkS) (width 0.127))
+    (fp_line (start -5.715 -2.54) (end -4.445 -2.54) (layer F.SilkS) (width 0.127))
+    (fp_line (start -4.445 -2.54) (end -3.81 -1.905) (layer F.SilkS) (width 0.127))
+    (fp_line (start -3.81 -1.905) (end -3.81 1.905) (layer F.SilkS) (width 0.127))
+    (fp_line (start -3.81 1.905) (end -4.445 2.54) (layer F.SilkS) (width 0.127))
+    (fp_line (start -4.445 2.54) (end -5.715 2.54) (layer F.SilkS) (width 0.127))
+    (pad 1 thru_hole circle (at -5.08 1.27) (size 1.6764 1.6764) (drill 1.016)
+      (layers *.Cu *.Mask F.SilkS)
+    )
+    (pad 2 thru_hole circle (at -5.08 -1.27) (size 1.6764 1.6764) (drill 1.016)
+      (layers *.Cu *.Mask F.SilkS)
+    )
+    (pad 3 thru_hole circle (at -2.54 1.27) (size 1.6764 1.6764) (drill 1.016)
+      (layers *.Cu *.Mask F.SilkS)
+    )
+    (pad 4 thru_hole circle (at -2.54 -1.27) (size 1.6764 1.6764) (drill 1.016)
+      (layers *.Cu *.Mask F.SilkS)
+    )
+    (pad 5 thru_hole circle (at 0 1.27) (size 1.6764 1.6764) (drill 1.016)
+      (layers *.Cu *.Mask F.SilkS)
+    )
+    (pad 6 thru_hole circle (at 0 -1.27) (size 1.6764 1.6764) (drill 1.016)
+      (layers *.Cu *.Mask F.SilkS)
+    )
+    (pad 7 thru_hole circle (at 2.54 1.27) (size 1.6764 1.6764) (drill 1.016)
+      (layers *.Cu *.Mask F.SilkS)
+    )
+    (pad 8 thru_hole circle (at 2.54 -1.27) (size 1.6764 1.6764) (drill 1.016)
+      (layers *.Cu *.Mask F.SilkS)
+    )
+    (pad 9 thru_hole circle (at 5.08 1.27) (size 1.6764 1.6764) (drill 1.016)
+      (layers *.Cu *.Mask F.SilkS)
+    )
+    (pad 10 thru_hole circle (at 5.08 -1.27) (size 1.6764 1.6764) (drill 1.016)
+      (layers *.Cu *.Mask F.SilkS)
+    )
+    (model ../3d_models/ab2_idc/AB2_HDR_M05-2V-S-3M.wrl
+      (at (xyz 0 0 0))
+      (scale (xyz 0.3937 0.3937 0.3937))
