File: template/ab2/ab2.kicad_pcb (KiCad board)
At the start: 2 copper layers, 0 parts

Commit message: template: changed soldermask width to 6mil
Other:
- rule solder_mask_min_width: 0.25 -> 0.1524
Changed lines of the file:
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@@
     (pad_drill 0.762)
     (pad_to_mask_clearance 0)
-    (solder_mask_min_width 0.25)
+    (solder_mask_min_width 0.1524)
     (aux_axis_origin 109.982 160.02)
     (grid_origin 109.982 160.02)
